File: anavi-play-phat.kicad_pcb (KiCad board)
At the start: 2 copper layers, 65 x 30 mm, 25 parts, among them U1 CAT24C32WI-GT3

Commit message: anavi-play-phat.kicad_pcb: Adjust buttons
Signed-off-by: Leon Anavi <leon@anavi.org>
Parts:
- moved < 0.41 mm to (150.1, 91.6)
- moved > 0.10 mm to (163.3, 91.6)
Routing:
- net GND: track 6.18 -> 0.00 mm, vias 1 -> 0
Changed lines of the file:
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@@
   (general
     (links 70)
-    (no_connects 10)
+    (no_connects 11)
     (area 136.817429 66.3 225.182572 110.000001)
     (thickness 1.6)
     (drawings 26)
-    (tracks 136)
+    (tracks 131)
     (zones 0)
     (modules 25)
@@
   )
   (module Buttons_Switches_ThroughHole:SW_PUSH_6mm_h4.3mm (layer F.Cu)
-    (at 150.114 91.186)
+    (at 150.114 91.5924)
     (descr "tactile push button, 6x6mm e.g. PHAP33xx series, height=4.3mm")
     (tags "tact sw push 6mm")
-    (fp_text reference < (at 8.5852 2.5908) (layer F.SilkS)
+    (fp_text reference < (at 8.5852 2.0828) (layer F.SilkS)
       (effects (font (size 2 1) (thickness 0.2)))
     )
@@
   )
   (module Buttons_Switches_ThroughHole:SW_PUSH_6mm_h4.3mm (layer F.Cu)
-    (at 163.322 91.694)
+    (at 163.322 91.5924)
     (descr "tactile push button, 6x6mm e.g. PHAP33xx series, height=4.3mm")
     (tags "tact sw push 6mm")
@@
     (descr "tactile push button, 6x6mm e.g. PHAP33xx series, height=4.3mm")
     (tags "tact sw push 6mm")
-    (fp_text reference A (at 3.3655 6.6675) (layer F.SilkS)
+    (fp_text reference A (at 3.3528 6.8072) (layer F.SilkS)
       (effects (font (size 1.2 1.2) (thickness 0.2)))
     )
@@
     (descr "tactile push button, 6x6mm e.g. PHAP33xx series, height=4.3mm")
     (tags "tact sw push 6mm")
-    (fp_text reference B (at 3.1623 6.604) (layer F.SilkS)
+    (fp_text reference B (at 3.1496 6.858) (layer F.SilkS)
       (effects (font (size 1.2 1.2) (thickness 0.2)))
     )
@@
     (effects (font (size 0.8 0.7) (thickness 0.125)))
   )
-  (gr_text "Made in Plovdiv, Bulgaria, EU" (at 212.598 89.916 90) (layer F.SilkS)
+  (gr_text "Made in Plovdiv, Bulgaria, EU" (at 212.4964 89.9668 90) (layer F.SilkS)
     (effects (font (size 0.8 0.8) (thickness 0.125)))
   )
@@
   (segment (start 209.97 84.89) (end 210 85) (width 0.5) (layer F.Cu) (net 1) (status 80000))
   (segment (start 210 88) (end 209.97 87.92) (width 0.5) (layer F.Cu) (net 1) (status 80000))
-  (segment (start 205.11 79.8) (end 206.2666 79.8) (width 0.5) (layer B.Cu) (net 2))
-  (segment (start 209.4566 82.99) (end 209.97 82.99) (width 0.5) (layer F.Cu) (net 2))
-  (segment (start 208.4832 82.0166) (end 209.4566 82.99) (width 0.5) (layer F.Cu) (net 2))
-  (via (at 208.4832 82.0166) (size 0.85) (drill 0.4) (layers F.Cu B.Cu) (net 2))
-  (segment (start 206.2666 79.8) (end 208.4832 82.0166) (width 0.5) (layer B.Cu) (net 2))
   (segment (start 156.85 77.26) (end 156.845 77.216) (width 0.5) (layer F.Cu) (net 3) (status 80000))
   (segment (start 156.85 77.26) (end 156.547 77.26) (width 0.5) (layer B.Cu) (net 3))
@@
   (segment (start 176.022 89.662) (end 181.102 89.662) (width 0.5) (layer F.Cu) (net 8))
   (segment (start 161.925 79.756) (end 161.93 79.8) (width 0.5) (layer B.Cu) (net 8) (status 80000))
-  (segment (start 156.614 91.186) (end 157.226 91.186) (width 0.5) (layer B.Cu) (net 9))
-  (segment (start 157.226 91.186) (end 161.036 87.376) (width 0.5) (layer B.Cu) (net 9))
+  (segment (start 156.614 91.5924) (end 157.226 91.5924) (width 0.5) (layer B.Cu) (net 9) (status 30))
+  (segment (start 157.226 91.5924) (end 161.036 87.376) (width 0.5) (layer B.Cu) (net 9) (status 10))
   (segment (start 161.036 87.376) (end 161.036 83.234) (width 0.5) (layer B.Cu) (net 9))
   (segment (start 161.036 83.234) (end 164.47 79.8) (width 0.5) (layer B.Cu) (net 9))
-  (segment (start 169.55 79.8) (end 169.55 91.422) (width 0.5) (layer B.Cu) (net 10))
-  (segment (start 169.55 91.422) (end 169.822 91.694) (width 0.5) (layer B.Cu) (net 10))
+  (segment (start 169.55 79.8) (end 169.55 91.3204) (width 0.5) (layer B.Cu) (net 10) (status 20))
+  (segment (start 169.55 91.3204) (end 169.822 91.5924) (width 0.5) (layer B.Cu) (net 10) (status 30))
   (segment (start 169.545 79.756) (end 169.55 79.8) (width 0.5) (layer F.Cu) (net 10) (status 80000))
   (segment (start 172.09 79.8) (end 172.09 97.531) (width 0.5) (layer B.Cu) (net 11))
